File: hardware/Solderin Station.kicad_pcb (KiCad board)
At the start: 2 copper layers, 95.9 x 129.5 mm, 72 parts, among them J1 ICSP, J10 9Vac, J11 ENCODER_MALE, J12 ENCODER_FEMALE, J13 BUTTON_FEMALE, J14 BUTTON_MALE, J15 LED_MALE, J16 LED_FEMALE, J17 LCD_I2C, J18 CONN_01X03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

Commit message: update firmware
Parts:
- C12: value 100n -> 10n
Changed lines of the file:
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@@
     (links 144)
     (no_connects 0)
-    (area 176.497857 23.369999 279.988334 153.5)
+    (area 182.804999 23.419999 278.840001 153.110001)
     (thickness 1.6)
     (drawings 40)
@@
       (effects (font (size 1 1) (thickness 0.15)))
     )
-    (fp_text value 100n (at 1.25 2.36 90) (layer F.Fab)
+    (fp_text value 10n (at 1.25 2.36 90) (layer F.Fab)
       (effects (font (size 1 1) (thickness 0.15)))
     )
@@
       (effects (font (size 1 1) (thickness 0.15)))
     )
-    (fp_text value ENCODER_MALE (at 2.54 3.81 90) (layer F.Fab)
+    (fp_text value ENCODER_MALE (at -1.905 -1.27 180) (layer F.Fab)
       (effects (font (size 1 1) (thickness 0.15)))
     )
@@
       (effects (font (size 1 1) (thickness 0.15)))
     )
-    (fp_text value BUTTON_MALE (at 1.27 3.81 90) (layer F.Fab)
+    (fp_text value BUTTON_MALE (at -1.905 -1.27 180) (layer F.Fab)
       (effects (font (size 1 1) (thickness 0.15)))
     )
@@
       (effects (font (size 1 1) (thickness 0.15)))
     )
-    (fp_text value LED_MALE (at 1.27 3.81 90) (layer F.Fab)
-      (effects (font (size 1 1) (thickness 0.15)))
-    )
+    (fp_text value LED_MALE (at -1.905 0.635 180) (layer F.Fab)
+      (effects (font (size 1 1) (thickness 0.15)))
+    )

Commit message: description is added in the .ino file
Parts:
- added C13: 100n, Capacitors_THT:C_Disc_D3.8mm_W2.6mm_P2.50mm, F.Cu at (227.3, 110.5)
- moved R9 6.35 mm to (229.9, 112.4)
Routing:
- net Net-(C13-Pad1): track 5.08 -> 15.3 mm
- net PTC+: track 21.6 -> 15.2 mm
