File: hardware/Solderin Station.sch (KiCad schematic (older format))
At the start: 68 parts, among them J1 ICSP, J10 9Vac, J11 ENCODER_MALE, J12 ENCODER_FEMALE, J13 BUTTON_FEMALE, J14 BUTTON_MALE, J15 LED_MALE, J16 LED_FEMALE, J17 LCD_I2C, J18 CONN_01X03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

Commit message: update firmware
Parts:
- C12: value 100n -> 10n
Changed lines of the file:
@@
 P 4300 5600
 F 0 "C12" H 4325 5700 50  0000 L CNN
-F 1 "100n" H 4325 5500 50  0000 L CNN
+F 1 "10n" H 4325 5500 50  0000 L CNN
 F 2 "Capacitors_THT:C_Disc_D3.8mm_W2.6mm_P2.50mm" H 4338 5450 50  0001 C CNN
 F 3 "" H 4300 5600 50  0001 C CNN

Commit message: description is added in the .ino file
Parts:
- added C13: 100n, Capacitors_THT:C_Disc_D3.8mm_W2.6mm_P2.50mm, symbol C
Connections:
- net GND: now also C13.2
- net at R10.2, R9.1, U6.2 (-): now also C13.1
Other:
- moved on the sheet: J13, J14, J3, J4, R9, SW2
